Commit message: Update URDF for new robot chassis and IMU frame in the iRob interface
Signed-off-by: TiNredmc <thipok17@gmail.com>

File: R1/description_r1/robot_core.xacro (robot description, xacro)
@@ -9,5 +9,5 @@
 		<parent link="base_link_r1"/>
 		<child link="chassis_r1"/>
-		<origin xyz="0.13 0 0"/>
+		<origin xyz="-0.1325 0 0"/>
 	</joint>
 	<link name="chassis_r1">
