Commit message: Updated dimension and lidar FoV for new probot model
Signed-off-by: TiNredmc <thipok17@gmail.com>

File: R1/description_r1/hokuyo.xacro (robot description, xacro)
@@ -2,5 +2,5 @@
 <robot xmlns:xacro="http://www.ros.org/wiki/xacro">
   <joint name="hokuyo_joint_r1" type="fixed">
-    <origin xyz="-0.265 0.0 0" rpy="3.141593 0.0 -3.141593" />
+    <origin xyz="-0.175 0.205 0" rpy="3.141593 0.0 2.356194" />
     <parent link="chassis_r1" />
     <child link="laser_frame_r1" />

File: R1/description_r1/robot_core.xacro (robot description, xacro)
@@ -9,5 +9,5 @@
 		<parent link="base_link_r1"/>
 		<child link="chassis_r1"/>
-		<origin xyz="0 0 0"/>
+		<origin xyz="0.13 0 0"/>
 	</joint>
 	<link name="chassis_r1">
@@ -15,5 +15,5 @@
 			<origin xyz="0 0 0.05"/>
 			<geometry>
-				<box size="0.54 0.54 0.12"/>
+				<box size="0.52 0.55 0.10"/>
 			</geometry>
 			<material name="white"/>

Commit message: Update to accomodate for two hokuyo lidar
Signed-off-by: TiNredmc <thipok17@gmail.com>

File: R1/description_r1/hokuyo.xacro (robot description, xacro)
@@ -4,7 +4,21 @@
     <origin xyz="-0.175 0.205 0" rpy="3.141593 0.0 2.356194" />
     <parent link="chassis_r1" />
-    <child link="laser_frame_r1" />
+    <child link="laser_frame1_r1" />
   </joint>
-  <link name="laser_frame_r1">
+  <link name="laser_frame1_r1">
+    <inertial>
+      <mass value="0.001" />
+      <origin xyz="0.0 0.0 0.0" />
+      <inertia ixx="0.0001" ixy="0.0" ixz="0.0"
+        iyy="0.0001" iyz="0.0"
+        izz="0.0001" />
+    </inertial>
+  </link>
+  <joint name="hokuyo_joint2_r1" type="fixed">
+    <origin xyz="0.26 0.12 0" rpy="0.0 0.0 0.0" />
+    <parent link="chassis_r1" />
+    <child link="laser_frame2_r1" />
+  </joint>
+  <link name="laser_frame2_r1">
     <inertial>
       <mass value="0.001" />
