Commit message: updated URDF to be more resemble the actual robot, TODO: use real Lidar RPY transform
Signed-off-by: TiNredmc <thipok17@gmail.com>

File: R1/description_r1/robot_core_r1.xacro (robot description, xacro)
@@ -14,4 +14,10 @@
 		<color rgba="0 0 0 1"/>
     </material>
+	<material name="red">
+		<color rgba="0.8 0.0 0.0 1"/>
+	</material>
+	<material name="green">
+		<color rgba="0.0 0.8 0.0 1"/>
+	</material>
     <!-- BASE LINK -->
     <link name="base_link_r1">
@@ -21,5 +27,5 @@
 		<parent link="base_link_r1"/>
 		<child link="chassis_r1"/>
-		<origin xyz="0 0 0"/>
+		<origin xyz="0 0 0.55"/>
 	</joint>
 	<link name="chassis_r1">
@@ -27,17 +33,17 @@
 			<origin xyz="0 0 0.1"/>
 			<geometry>
-				<box size="0.5 0.5 0.03"/>
-			</geometry>
-			<material name="white"/>
-		</visual>
-		<collision>
-			<origin xyz="0 0 0.1"/>
-			<geometry>
-				<box size="0.5 0.5 0.03"/>
-			</geometry>
-		</collision>
-		<xacro:inertial_box mass="0.2" x="0.5" y="0.5" z="0.03">
-        	<origin xyz="0 0 0.1" rpy="0 0 0"/>
-    	</xacro:inertial_box>
+				<cylinder radius="0.4" length="1.2"/>
+			</geometry>
+			<material name="green"/>
+		</visual>
+		<collision>
+			<origin xyz="0 0 0.2"/>
+			<geometry>
+				<cylinder radius="0.4" length="1.2"/>
+			</geometry>
+		</collision>
+		<xacro:inertial_cylinder mass="25.0" radius="0.4" length="1.2">
+        	<origin xyz="0 0 -0.6" rpy="0 0 0"/>
+    	</xacro:inertial_cylinder>
 	</link>
 	<gazebo reference="chassis_r1">
@@ -152,5 +158,5 @@
 		<mu2 value="0.5"/>
     </gazebo>
-	<link name="lidar_link_1_r1">
+    <link name="lidar_link_1_r1">
     <inertial>
       <origin xyz="0 0 0" rpy="0 0 0"/>
@@ -158,10 +164,4 @@
       <inertia ixx="0.001"  ixy="0"  ixz="0" iyy="0.001" iyz="0" izz="0.001" />
     </inertial>
-    <collision>
-      <origin xyz="0 0 0" rpy="0 0 0"/>
-      <geometry>
-         <cylinder radius="0.0508" length="0.055"/>
-      </geometry>
-    </collision>
     <visual>
       <origin xyz="0 0 0" rpy="0 0 0"/>
@@ -174,5 +174,5 @@
     <parent link="base_link_r1"/>
     <child link="lidar_link_1_r1"/>
-    <origin xyz="0.265 0 0.03" rpy="0 0 0"/>
+    <origin xyz="0.35 0 0.03" rpy="0 0 0"/>
   </joint>
   <gazebo reference="lidar_link_1_r1">
@@ -215,10 +215,4 @@
       <inertia ixx="0.001"  ixy="0"  ixz="0" iyy="0.001" iyz="0" izz="0.001" />
     </inertial>
-    <collision>
-      <origin xyz="0 0 0" rpy="0 0 0"/>
-      <geometry>
-         <cylinder radius="0.0508" length="0.055"/>
-      </geometry>
-    </collision>
     <visual>
       <origin xyz="0 0 0" rpy="0 0 0"/>
@@ -231,5 +225,5 @@
     <parent link="base_link_r1"/>
     <child link="lidar_link_2_r1"/>
-	<origin xyz="-0.265 0 0.03" rpy="0 0 3.141593"/>
+	<origin xyz="-0.35 0 0.03" rpy="0 0 3.141593"/>
   </joint>
   <gazebo reference="lidar_link_2_r1">

File: R2/description_r2/robot_core_r2.xacro (robot description, xacro)
@@ -14,4 +14,10 @@
 		<color rgba="0 0 0 1"/>
     </material>
+	<material name="red">
+		<color rgba="0.8 0.0 0.0 1"/>
+	</material>
+	<material name="green">
+		<color rgba="0.0 0.8 0.0 1"/>
+	</material>
     <!-- BASE LINK -->
     <link name="base_link_r2">
@@ -21,5 +27,5 @@
 		<parent link="base_link_r2"/>
 		<child link="chassis_r2"/>
-		<origin xyz="0 0 0"/>
+		<origin xyz="0 0 0.55"/>
 	</joint>
 	<link name="chassis_r2">
@@ -27,17 +33,17 @@
 			<origin xyz="0 0 0.1"/>
 			<geometry>
-				<box size="0.5 0.5 0.03"/>
-			</geometry>
-			<material name="white"/>
-		</visual>
-		<collision>
-			<origin xyz="0 0 0.1"/>
-			<geometry>
-				<box size="0.5 0.5 0.03"/>
-			</geometry>
-		</collision>
-		<xacro:inertial_box mass="0.2" x="0.5" y="0.5" z="0.03">
-        	<origin xyz="0 0 0.1" rpy="0 0 0"/>
-    	</xacro:inertial_box>
+				<cylinder radius="0.4" length="1.2"/>
+			</geometry>
+			<material name="red"/>
+		</visual>
+		<collision>
+			<origin xyz="0 0 0.2"/>
+			<geometry>
+				<cylinder radius="0.4" length="1.2"/>
+			</geometry>
+		</collision>
+		<xacro:inertial_cylinder mass="25.0" radius="0.4" length="1.2">
+        	<origin xyz="0 0 -0.6" rpy="0 0 0"/>
+    	</xacro:inertial_cylinder>
 	</link>
 	<gazebo reference="chassis_r2">
@@ -174,5 +180,5 @@
     <parent link="base_link_r2"/>
     <child link="lidar_link_1_r2"/>
-    <origin xyz="0.265 0 0.03" rpy="0 0 0"/>
+    <origin xyz="0.35 0 0.03" rpy="0 0 0"/>
   </joint>
   <gazebo reference="lidar_link_1_r2">
@@ -231,5 +237,5 @@
     <parent link="base_link_r2"/>
     <child link="lidar_link_2_r2"/>
-	<origin xyz="-0.265 0 0.03" rpy="0 0 3.141593"/>
+	<origin xyz="-0.35 0 0.03" rpy="0 0 3.141593"/>
   </joint>
   <gazebo reference="lidar_link_2_r2">
