Commit message: updated file for R2
Signed-off-by: TiNredmc <thipok17@gmail.com>

File: R2/description_r2/asus_xtion.xacro (robot description, xacro)
@@ -1,11 +1,11 @@
 <?xml version="1.0"?>
 <robot xmlns:xacro="http://www.ros.org/wiki/xacro">
-  <joint name="base_camera_joint_r2" type="fixed">
+  <joint name="base_camera_joint" type="fixed">
     <origin xyz="0.112 0 0.1605"
             rpy="1.5708 3.1415 1.5708" />
-    <parent link="chassis_r2" />
-    <child link="camera_link_r2" />
+    <parent link="chassis" />
+    <child link="camera_link" />
   </joint>
-  <link name="camera_link_r2">
+  <link name="camera_link">
     <inertial>
       <mass value="0.01" />
@@ -28,10 +28,10 @@
     </collision>
   </link>
-  <joint name="camera_depth_optical_joint_r2" type="fixed">
+  <joint name="camera_depth_optical_joint" type="fixed">
     <origin xyz="-0.04 0 0" rpy="3.1415 3.1415 3.1415" />
-    <parent link="camera_link_r2" />
-    <child link="openni_depth_optical_frame_r2" />
+    <parent link="camera_link" />
+    <child link="openni_depth_optical_frame" />
   </joint>
-  <link name="openni_depth_optical_frame_r2">
+  <link name="openni_depth_optical_frame">
     <inertial>
       <mass value="0.001" />
@@ -42,10 +42,10 @@
     </inertial>
   </link>
- <joint name="laser_joint_r2" type="fixed">
+ <joint name="laser_joint" type="fixed">
     <origin xyz="-0.31 -0.15 0" rpy="0.0 0.0 -3.1415" />
-    <parent link="chassis_r2" />
-    <child link="laser_frame_r2" />
+    <parent link="chassis" />
+    <child link="laser_frame" />
   </joint>
-  <link name="laser_frame_r2">
+  <link name="laser_frame">
     <inertial>
       <mass value="0.001" />

File: R2/description_r2/robot.urdf.xacro (robot description, xacro)
@@ -2,4 +2,5 @@
 <robot xmlns:xacro="http://www.ros.org/wiki/xacro"  name="robot">
     <xacro:include filename="robot_core.xacro" />
-    <xacro:include filename="asus_xtion.xacro" />
+    <xacro:include filename="imu.xacro" />
+    <xacro:include filename="hokuyo.xacro" />
 </robot>

File: R2/description_r2/robot_core.xacro (robot description, xacro)
@@ -9,5 +9,5 @@
 		<parent link="base_link_r2"/>
 		<child link="chassis_r2"/>
-		<origin xyz="0 0 0"/>
+		<origin xyz="-0.1325 0 0"/>
 	</joint>
 	<link name="chassis_r2">
@@ -15,5 +15,5 @@
 			<origin xyz="0 0 0.05"/>
 			<geometry>
-				<box size="0.54 0.54 0.12"/>
+				<box size="0.52 0.55 0.10"/>
 			</geometry>
 			<material name="white"/>
